File: report/schematic/schematic.kicad_sch (KiCad schematic)
At the start: 7 parts, among them P1 P, P2 P, SW1 Push_Button, SW2 Push_Button, U1 ESP32-DevKitM-1, U2 MAX7219

Commit message: update report
Parts:
- added BZ1: Buzzer_5V, Buzzer_Beeper:MagneticBuzzer_ProSignal_ABT-410-RC, symbol PCM_SL_Devices:Buzzer_5V
Connections:
- net at P1.3 (c), P2.3 (c), SW1.1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: now also BZ1.2
- net at SW2.2: now also U1.29 (GPIO19); no longer U1.31 (GPIO21)
- net at U1.10 (32K_XP/GPIO32/ADC1_CH4): now also BZ1.1
- net at U1.11 (32K_XN/GPIO33/ADC1_CH5): now also P1.2 (b)
- net at U1.9 (GPIO35/ADC1_CH7): now also P2.2 (b)
Changed lines of the file:
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@@
+	)
+	(junction
+		(at 106.68 109.22)
+		(diameter 0)
+		(color 0 0 0 0)
 	)
 	(junction
@@
 	(wire
 		(pts
+			(xy 15.24 127) (xy 15.24 66.04)
+		)
+		(stroke
+			(width 0)
+			(type default)
+		)
+	)
+	(wire
+		(pts
 			(xy 120.65 55.88) (xy 120.65 111.76)
 		)
@@
 	(wire
 		(pts
+			(xy 15.24 66.04) (xy 24.13 66.04)
+		)
+		(stroke
+			(width 0)
+			(type default)
+		)
+	)
+	(wire
+		(pts
 			(xy 43.18 109.22) (xy 57.15 109.22)
 		)
@@
 	(wire
 		(pts
+			(xy 90.17 72.39) (xy 99.06 72.39)
+		)
+		(stroke
+			(width 0)
+			(type default)
+		)
+	)
+	(wire
+		(pts
 			(xy 158.75 33.02) (xy 158.75 73.66)
 		)
@@
 	(wire
 		(pts
+			(xy 49.53 129.54) (xy 49.53 127)
+		)
+		(stroke
+			(width 0)
+			(type default)
+		)
+	)
+	(wire
+		(pts
 			(xy 128.27 50.8) (xy 116.84 50.8)
 		)
@@
 	(wire
 		(pts
+			(xy 106.68 109.22) (xy 119.38 109.22)
+		)
+		(stroke
+			(width 0)
+			(type default)
+		)
+	)
+	(wire
+		(pts
 			(xy 124.46 134.62) (xy 160.02 134.62)
 		)
@@
 	(wire
 		(pts
+			(xy 24.13 60.96) (xy 13.97 60.96)
+		)
+		(stroke
+			(width 0)
+			(type default)
+		)
+	)
+	(wire
+		(pts
 			(xy 20.32 85.09) (xy 20.32 114.3)
 		)
@@
 	(wire
 		(pts
+			(xy 16.51 29.21) (xy 96.52 29.21)
+		)
+		(stroke
+			(width 0)
+			(type default)
+		)
+	)
+	(wire
+		(pts
+			(xy 99.06 72.39) (xy 99.06 128.27)
+		)
+		(stroke
+			(width 0)
+			(type default)
+		)
+	)
+	(wire
+		(pts
 			(xy 193.04 60.96) (xy 193.04 78.74)
 		)
@@
 	(wire
 		(pts
+			(xy 16.51 63.5) (xy 16.51 29.21)
+		)
+		(stroke
+			(width 0)
+			(type default)
+		)
+	)
+	(wire
+		(pts
 			(xy 25.4 124.46) (xy 30.48 124.46)
 		)
@@
 	(wire
 		(pts
-			(xy 99.06 74.93) (xy 99.06 128.27)
-		)
-		(stroke
-			(width 0)
-			(type default)
-		)
-	)
-	(wire
-		(pts
 			(xy 24.13 85.09) (xy 20.32 85.09)
 		)
@@
 	(wire
 		(pts
+			(xy 24.13 63.5) (xy 16.51 63.5)
+		)
+		(stroke
+			(width 0)
+			(type default)
+		)
+	)
+	(wire
+		(pts
 			(xy 116.84 50.8) (xy 116.84 96.52)
 		)
@@
 	(wire
 		(pts
+			(xy 96.52 29.21) (xy 96.52 54.61)
+		)
+		(stroke
+			(width 0)
+			(type default)
+		)
+	)
+	(wire
+		(pts
 			(xy 24.13 77.47) (xy 17.78 77.47)
 		)
@@
 	(wire
 		(pts
+			(xy 30.48 127) (xy 15.24 127)
+		)
+		(stroke
+			(width 0)
+			(type default)
+		)
+	)
+	(wire
+		(pts
 			(xy 118.11 104.14) (xy 160.02 104.14)
 		)
@@
 	(wire
 		(pts
+			(xy 13.97 60.96) (xy 13.97 129.54)
+		)
+		(stroke
+			(width 0)
+			(type default)
+		)
+	)
+	(wire
+		(pts
+			(xy 106.68 54.61) (xy 106.68 109.22)
+		)
+		(stroke
+			(width 0)
+			(type default)
+		)
+	)
+	(wire
+		(pts
 			(xy 156.21 71.12) (xy 157.48 71.12)
 		)
@@
 	(wire
 		(pts
-			(xy 86.36 109.22) (xy 119.38 109.22)
+			(xy 86.36 109.22) (xy 106.68 109.22)
 		)
 		(stroke
@@
 	(wire
 		(pts
+			(xy 13.97 129.54) (xy 49.53 129.54)
+		)
+		(stroke
+			(width 0)
+			(type default)
+		)
+	)
+	(wire
+		(pts
 			(xy 119.38 109.22) (xy 119.38 73.66)
 		)
@@
 		(pts
 			(xy 86.36 109.22) (xy 86.36 128.27)
-		)
-		(stroke
-			(width 0)
-			(type default)
-		)
-	)
-	(wire
-		(pts
-			(xy 90.17 74.93) (xy 99.06 74.93)
 		)
 		(stroke
@@
 	)
 	(symbol
+		(lib_id "PCM_SL_Devices:Buzzer_5V")
+		(at 101.6 54.61 0)
+		(unit 1)
+		(exclude_from_sim no)
+		(in_bom yes)
+		(on_board yes)
+		(dnp no)
+		(fields_autoplaced yes)
+		(property "Reference" "BZ1"
+			(at 101.6 46.99 0)
+			(effects
+				(font
+					(size 1.27 1.27)
+				)
+			)
+		)
+		(property "Value" "Buzzer_5V"
+			(at 101.6 49.53 0)
+			(effects
+				(font
+					(size 1.27 1.27)
+				)
+			)
+		)
+		(property "Footprint" "Buzzer_Beeper:MagneticBuzzer_ProSignal_ABT-410-RC"
+			(at 101.6 44.45 0)
+			(effects
+				(font
+					(size 1.27 1.27)
+				)
+				(hide yes)
+			)
+		)
+		(property "Datasheet" ""
+			(at 101.6 46.99 0)
+			(effects
+				(font
+					(size 1.27 1.27)
+				)
+				(hide yes)
+			)
+		)
+		(property "Description" "Buzzer 5V"
+			(at 101.6 54.61 0)
+			(effects
+				(font
+					(size 1.27 1.27)
+				)
+				(hide yes)
+			)
+		)
+		(pin "2"
+		)
+		(pin "1"
+		)
+		(instances
+			(project ""
+				(path "/6f2be3e6-940b-4a2d-a82a-4b02fef2fa63"
+					(reference "BZ1")
+					(unit 1)
+				)
+			)
+		)
+	)
+	(symbol
 		(lib_id "PCM_Espressif:ESP32-DevKitM-1")
 		(at 57.15 73.66 0)
@@
 	)
 	(symbol
-		(lib_name "PCM_Elektuur_1:P")
 		(lib_id "PCM_Elektuur_1:P")
 		(at 35.56 124.46 270)
@@
 	)
 	(symbol
-		(lib_name "PCM_Elektuur_1:P")
 		(lib_id "PCM_Elektuur_1:P")
 		(at 54.61 124.46 270)
